Commit message: Add gazebo sim

File: jetson/sp8_ws/src/sp8_robot/description/sp8.urdf.xacro (robot description, xacro)
@@ -2,3 +2,4 @@
 <robot xmlns:xacro="http://www.ros.org/wiki/xacro" name="sp8">
     <xacro:include filename="sp8_core.xacro"/>
+    <xacro:include filename="gazebo_control.xacro"/>
 </robot>

File: jetson/sp8_ws/src/sp8_robot/description/sp8_core.xacro (robot description, xacro)
@@ -15,5 +15,5 @@
         <parent link="base_footprint_link"/>
         <child link="base_link"/>
-        <origin xyz="0.0 0.0 0.052"/>
+        <origin xyz="0.0 0.0 0.052"/> <!-- 0.052-->
     </joint>
     <link name="base_link">
@@ -31,5 +31,5 @@
             </geometry>
         </collision>
-        <xacro:inertial_cylinder mass = "2.0" length = "0.1" radius = "0.125">
+        <xacro:inertial_cylinder mass = "3.0" length = "0.1" radius = "0.125">
             <origin xyz="0.0 0.0 0.036" rpy="0.0 0.0 0.0"/>
         </xacro:inertial_cylinder>
@@ -39,23 +39,25 @@
     </gazebo>
     <!-- LEFT WHEEL LINK -->
-    <joint name="left_wheel_join" type="continuous">
+    <joint name="left_wheel_joint" type="continuous">
         <parent link="base_link"/>
         <child link="left_wheel_link"/>
-        <origin xyz="0.0 0.08 0.0" rpy="-${pi/2} 0.0 0.0"/>
-        <axis xyz="0.0 0.0 1.0"/>
+        <origin xyz="0.0 0.08 0.0" rpy="0.0 0.0 0.0"/>
+        <axis xyz="0.0 1.0 0.0"/>
     </joint>
     <link name="left_wheel_link">
         <visual>
+            <origin rpy= "1.5707 0.0 0.0"/>
             <geometry>
-                <cylinder radius="0.0515" length="0.005"/>
+                <cylinder radius="0.053" length="0.005"/>
             </geometry>
             <material name="black"/>
         </visual>
         <collision>
+            <origin rpy= "1.5707 0.0 0.0"/>
             <geometry>
-                <cylinder radius="0.0515" length="0.005"/>
+                <cylinder radius="0.053" length="0.005"/>
             </geometry>
         </collision>
-        <xacro:inertial_cylinder mass = "0.01" length = "0.005" radius = "0.0515">
+        <xacro:inertial_cylinder mass = "0.01" length = "0.005" radius = "0.053">
             <origin xyz="0.0 0.0 0.0" rpy="0.0 0.0 0.0"/>
         </xacro:inertial_cylinder>
@@ -63,25 +65,29 @@
     <gazebo reference="left_wheel_link">
         <material>Gazebo/Black</material>
+        <mu1 value="1.0"/>
+        <mu2 value="1.0"/>
     </gazebo>
     <!-- RIGHT WHEEL LINK -->
-    <joint name="right_wheel_join" type="continuous">
+    <joint name="right_wheel_joint" type="continuous">
         <parent link="base_link"/>
         <child link="right_wheel_link"/>
-        <origin xyz="0.0 -0.08 0.0" rpy="${pi/2} 0.0 0.0"/>
-        <axis xyz="0.0 0.0 -1.0"/>
+        <origin xyz="0.0 -0.08 0.0" rpy="0.0 0.0 0.0"/>
+        <axis xyz="0.0 1.0 0.0"/>
     </joint>
     <link name="right_wheel_link">
         <visual>
+            <origin rpy= "1.5707 0.0 0.0"/>
             <geometry>
-                <cylinder radius="0.0515" length="0.005"/>
+                <cylinder radius="0.053" length="0.005"/>
             </geometry>
             <material name="black"/>
         </visual>
         <collision>
+            <origin rpy= "1.5707 0.0 0.0"/>
             <geometry>
-                <cylinder radius="0.0515" length="0.005"/>
+                <cylinder radius="0.053" length="0.005"/>
             </geometry>
         </collision>
-        <xacro:inertial_cylinder mass = "0.01" length = "0.005" radius = "0.0515">
+        <xacro:inertial_cylinder mass = "0.01" length = "0.005" radius = "0.053">
             <origin xyz="0.0 0.0 0.0" rpy="0.0 0.0 0.0"/>
         </xacro:inertial_cylinder>
@@ -89,4 +95,6 @@
     <gazebo reference="right_wheel_link">
         <material>Gazebo/Black</material>
+        <mu1 value="1.0"/>
+        <mu2 value="1.0"/>
     </gazebo>
     <!-- FRONT CASTER LINK -->
@@ -98,5 +106,5 @@
     <link name="front_caster_link">
         <visual>
-            <origin xyz="0.0 0.0 -0.026"/>
+            <origin xyz="0.0 0.0 -0.01"/> <!--0.26-->
             <geometry>
                 <cylinder radius="0.0125" length="0.052"/>
@@ -116,4 +124,6 @@
     <gazebo reference="front_caster_link">
         <material>Gazebo/Black</material>
+        <mu1 value="0.001"/>
+        <mu2 value="0.001"/>
     </gazebo>
     <!-- BACK CASTER LINK -->
@@ -125,5 +135,5 @@
     <link name="back_caster_link">
         <visual>
-            <origin xyz="0.0 0.0 -0.026"/>
+            <origin xyz="0.0 0.0 -0.01"/> <!--0.26-->
             <geometry>
                 <cylinder radius="0.025" length="0.052"/>
@@ -143,4 +153,6 @@
     <gazebo reference="back_caster_link">
         <material>Gazebo/White</material>
+        <mu1 value="0.001"/>
+        <mu2 value="0.001"/>
     </gazebo>
 </robot>
