Commit message: Add bringup

File: jetson/sp8_ws/src/sp8_robot/description/sp8_core.xacro (robot description, xacro)
@@ -9,9 +9,9 @@
     </material>
     <!-- BASE FOOTPRINT LINK-->
-    <link name="base_footprint_link">
+    <link name="base_footprint">
     </link>
     <!-- BASE LINK -->
-    <joint name="base_link_join" type="fixed">
-        <parent link="base_footprint_link"/>
+    <joint name="base_link_joint" type="fixed">
+        <parent link="base_footprint"/>
         <child link="base_link"/>
         <origin xyz="0.0 0.0 0.052"/> <!-- 0.052-->
